File: pmod/RotaryEncoder/KiCad/RotaryEncoder/RotaryEncoder.kicad_sch (KiCad schematic)
At the start: 15 parts, among them J1 Conn_01x06, U1 PEC11R-4325F-S0012

Commit message: work in progress
Connections:
- net A: now also C1.2, R3.2; no longer R1.2, R3.1, U1.A1 (A_CHANNEL)
- net B: now also C2.2, R4.1; no longer R2.2, R4.2, U1.B1 (B_CHANNEL)
- net BTN: now also C3.1, R6.2; no longer R5.1, R6.1, U1.1 (COM)
- new net: R5.1, R6.1, U1.1 (COM)
- new net: R2.2, R4.2, U1.B1 (B_CHANNEL)
- new net: R1.2, R3.1, U1.A1 (A_CHANNEL)
Other:
- moved on the sheet: C3, R5, R6
Changed lines of the file:
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@@
 	)
 	(junction
-		(at 63.5 69.85)
+		(at 55.88 41.91)
 		(diameter 0)
 		(color 0 0 0 0)
@@
 	)
 	(junction
-		(at 63.5 41.91)
+		(at 137.16 60.96)
 		(diameter 0)
 		(color 0 0 0 0)
 	)
 	(junction
-		(at 127 66.04)
+		(at 63.5 41.91)
 		(diameter 0)
 		(color 0 0 0 0)
@@
 	)
 	(junction
+		(at 55.88 69.85)
+		(diameter 0)
+		(color 0 0 0 0)
+	)
+	(junction
 		(at 127 54.61)
 		(diameter 0)
@@
 	(wire
 		(pts
-			(xy 63.5 59.69) (xy 63.5 69.85)
+			(xy 137.16 60.96) (xy 137.16 63.5)
 		)
 		(stroke
@@
 	(wire
 		(pts
-			(xy 63.5 41.91) (xy 63.5 50.8)
+			(xy 63.5 59.69) (xy 63.5 69.85)
 		)
 		(stroke
@@
 	(wire
 		(pts
-			(xy 130.81 66.04) (xy 127 66.04)
+			(xy 63.5 41.91) (xy 63.5 50.8)
 		)
 		(stroke
@@
 	(wire
 		(pts
-			(xy 62.23 41.91) (xy 63.5 41.91)
+			(xy 128.27 60.96) (xy 127 60.96)
 		)
 		(stroke
@@
 	(wire
 		(pts
-			(xy 63.5 59.69) (xy 78.74 59.69)
+			(xy 135.89 60.96) (xy 137.16 60.96)
 		)
 		(stroke
@@
 	(wire
 		(pts
-			(xy 63.5 38.1) (xy 63.5 41.91)
+			(xy 62.23 41.91) (xy 63.5 41.91)
 		)
 		(stroke
@@
 	(wire
 		(pts
-			(xy 78.74 57.15) (xy 76.2 57.15)
+			(xy 63.5 59.69) (xy 78.74 59.69)
 		)
 		(stroke
@@
 	(wire
 		(pts
-			(xy 127 54.61) (xy 127 66.04)
+			(xy 55.88 38.1) (xy 55.88 41.91)
 		)
 		(stroke
@@
 	(wire
 		(pts
-			(xy 78.74 54.61) (xy 77.47 54.61)
+			(xy 78.74 57.15) (xy 76.2 57.15)
 		)
 		(stroke
@@
 	(wire
 		(pts
-			(xy 63.5 69.85) (xy 63.5 73.66)
+			(xy 127 54.61) (xy 127 60.96)
 		)
 		(stroke
@@
 	(wire
 		(pts
-			(xy 77.47 54.61) (xy 77.47 50.8)
+			(xy 78.74 54.61) (xy 77.47 54.61)
 		)
 		(stroke
@@
 	(wire
 		(pts
-			(xy 127 54.61) (xy 132.08 54.61)
+			(xy 128.27 54.61) (xy 127 54.61)
 		)
 		(stroke
@@
 	(wire
 		(pts
-			(xy 127 66.04) (xy 127 69.85)
+			(xy 55.88 69.85) (xy 55.88 73.66)
 		)
 		(stroke
@@
 	(wire
 		(pts
-			(xy 77.47 50.8) (xy 63.5 50.8)
+			(xy 137.16 60.96) (xy 138.43 60.96)
 		)
 		(stroke
@@
 		)
 	)
+	(wire
+		(pts
+			(xy 77.47 54.61) (xy 77.47 50.8)
+		)
+		(stroke
+			(width 0)
+			(type default)
+		)
+	)
+	(wire
+		(pts
+			(xy 77.47 50.8) (xy 63.5 50.8)
+		)
+		(stroke
+			(width 0)
+			(type default)
+		)
+	)
 	(global_label "A"
 		(shape input)
@@
 	(global_label "A"
 		(shape output)
-		(at 63.5 38.1 90)
+		(at 55.88 38.1 90)
 		(fields_autoplaced yes)
 		(effects
@@
 		)
 		(property "Intersheetrefs" "${INTERSHEET_REFS}"
-			(at 63.5 34.0262 90)
+			(at 55.88 34.0262 90)
 			(effects
 				(font
@@
 	(global_label "BTN"
 		(shape output)
-		(at 127 69.85 270)
+		(at 137.16 63.5 270)
 		(fields_autoplaced yes)
 		(effects
@@
 		)
 		(property "Intersheetrefs" "${INTERSHEET_REFS}"
-			(at 127 76.4033 90)
+			(at 137.16 70.0533 90)
 			(effects
 				(font
@@
 	(global_label "B"
 		(shape output)
-		(at 63.5 73.66 270)
+		(at 55.88 73.66 270)
 		(fields_autoplaced yes)
 		(effects
@@
 		)
 		(property "Intersheetrefs" "${INTERSHEET_REFS}"
-			(at 63.5 77.9152 90)
+			(at 55.88 77.9152 90)
 			(effects
 				(font
@@
 	(symbol
 		(lib_id "power:GND")
-		(at 146.05 66.04 90)
+		(at 146.05 60.96 90)
 		(unit 1)
 		(exclude_from_sim no)
@@
 		(fields_autoplaced yes)
 		(property "Reference" "#PWR010"
-			(at 152.4 66.04 0)
+			(at 152.4 60.96 0)
 			(effects
 				(font
@@
 		)
 		(property "Value" "GND"
-			(at 149.86 66.0401 90)
+			(at 149.86 60.9601 90)
 			(effects
 				(font
@@
 		)
 		(property "Footprint" ""
-			(at 146.05 66.04 0)
+			(at 146.05 60.96 0)
 			(effects
 				(font
@@
 		)
 		(property "Datasheet" ""
-			(at 146.05 66.04 0)
+			(at 146.05 60.96 0)
 			(effects
 				(font
@@
 		)
 		(property "Description" "Power symbol creates a global label with name \"GND\" , ground"
-			(at 146.05 66.04 0)
+			(at 146.05 60.96 0)
 			(effects
 				(font
@@
 	(symbol
 		(lib_id "Device:R")
-		(at 134.62 66.04 90)
+		(at 132.08 60.96 90)
 		(unit 1)
 		(exclude_from_sim no)
@@
 		(fields_autoplaced yes)
 		(property "Reference" "R6"
-			(at 134.62 72.39 90)
+			(at 132.08 67.31 90)
 			(effects
 				(font
@@
 		)
 		(property "Value" "10K"
-			(at 134.62 69.85 90)
+			(at 132.08 64.77 90)
 			(effects
 				(font
@@
 		)
 		(property "Footprint" "Resistor_THT:R_Axial_DIN0204_L3.6mm_D1.6mm_P5.08mm_Horizontal"
-			(at 134.62 67.818 90)
+			(at 132.08 62.738 90)
 			(effects
 				(font
@@
 		)
 		(property "Datasheet" "~"
-			(at 134.62 66.04 0)
+			(at 132.08 60.96 0)
 			(effects
 				(font
@@
 		)
 		(property "Description" "Resistor"
-			(at 134.62 66.04 0)
+			(at 132.08 60.96 0)
 			(effects
 				(font
@@
 	(symbol
 		(lib_id "Device:C")
-		(at 142.24 66.04 90)
+		(at 142.24 60.96 90)
 		(unit 1)
 		(exclude_from_sim no)
@@
 		(fields_autoplaced yes)
 		(property "Reference" "C3"
-			(at 143.5101 69.85 0)
+			(at 143.5101 64.77 0)
 			(effects
 				(font
@@
 		)
 		(property "Value" "0.01uF"
-			(at 140.9701 69.85 0)
+			(at 140.9701 64.77 0)
 			(effects
 				(font
@@
 		)
 		(property "Footprint" "Capacitor_THT:C_Disc_D3.8mm_W2.6mm_P2.50mm"
-			(at 146.05 65.0748 0)
+			(at 146.05 59.9948 0)
 			(effects
 				(font
@@
 		)
 		(property "Datasheet" "~"
-			(at 142.24 66.04 0)
+			(at 142.24 60.96 0)
 			(effects
 				(font
@@
 		)
 		(property "Description" "Unpolarized capacitor"
-			(at 142.24 66.04 0)
+			(at 142.24 60.96 0)
 			(effects
 				(font
@@
 	(symbol
 		(lib_id "Device:R")
-		(at 135.89 54.61 90)
+		(at 132.08 54.61 90)
 		(unit 1)
 		(exclude_from_sim no)
@@
 		(dnp no)
 		(property "Reference" "R5"
-			(at 134.874 52.07 90)
+			(at 131.064 52.07 90)
 			(effects
 				(font
@@
 		)
 		(property "Value" "10K"
-			(at 134.6201 57.15 90)
+			(at 130.8101 57.15 90)
 			(effects
 				(font
@@
 		)
 		(property "Footprint" "Resistor_THT:R_Axial_DIN0204_L3.6mm_D1.6mm_P5.08mm_Horizontal"
-			(at 135.89 56.388 90)
+			(at 132.08 56.388 90)
 			(effects
 				(font
@@
 		)
 		(property "Datasheet" "~"
+			(at 132.08 54.61 0)
+			(effects
+				(font
+					(size 1.27 1.27)
+				)
+				(hide yes)
+			)
+		)
+		(property "Description" "Resistor"
+			(at 132.08 54.61 0)
+			(effects
+				(font
+					(size 1.27 1.27)
+				)
+				(hide yes)
+			)
+		)
+		(pin "1"
+		)
+		(pin "2"
+		)
+		(instances
+			(project "RotaryEncoder"
+				(path "/4e64649f-140d-4c43-8072-32119b91f969"
+					(reference "R5")
+					(unit 1)
+				)
+			)
+		)
+	)
+	(symbol
+		(lib_id "power:VCC")
+		(at 135.89 54.61 270)
+		(unit 1)
+		(exclude_from_sim no)
+		(in_bom yes)
+		(on_board yes)
+		(dnp no)
+		(property "Reference" "#PWR02"
+			(at 132.08 54.61 0)
+			(effects
+				(font
+					(size 1.27 1.27)
+				)
+				(hide yes)
+			)
+		)
+		(property "Value" "VCC"
+			(at 140.97 54.61 90)
+			(effects
+				(font
+					(size 1.27 1.27)
+				)
+			)
+		)
+		(property "Footprint" ""
 			(at 135.89 54.61 0)
 			(effects
@@
 			)
 		)
-		(property "Description" "Resistor"
+		(property "Datasheet" ""
 			(at 135.89 54.61 0)
 			(effects
@@
 			)
 		)
-		(pin "1"
-		)
-		(pin "2"
-		)
-		(instances
-			(project "RotaryEncoder"
-				(path "/4e64649f-140d-4c43-8072-32119b91f969"
-					(reference "R5")
-					(unit 1)
-				)
-			)
-		)
-	)
-	(symbol
-		(lib_id "power:VCC")
-		(at 139.7 54.61 270)
-		(unit 1)
-		(exclude_from_sim no)
-		(in_bom yes)
-		(on_board yes)
-		(dnp no)
-		(property "Reference" "#PWR02"
+		(property "Description" "Power symbol creates a global label with name \"VCC\""
 			(at 135.89 54.61 0)
 			(effects
 				(font
-					(size 1.27 1.27)
-				)
-				(hide yes)
-			)
-		)
-		(property "Value" "VCC"
-			(at 144.78 54.61 90)
-			(effects
-				(font
-					(size 1.27 1.27)
-				)
-			)
-		)
-		(property "Footprint" ""
-			(at 139.7 54.61 0)
-			(effects
-				(font
-					(size 1.27 1.27)
-				)
-				(hide yes)
-			)
-		)
-		(property "Datasheet" ""
-			(at 139.7 54.61 0)
-			(effects
-				(font
-					(size 1.27 1.27)
-				)
-				(hide yes)
-			)
-		)
-		(property "Description" "Power symbol creates a global label with name \"VCC\""
-			(at 139.7 54.61 0)
-			(effects
-				(font
