File: pmod/RotaryEncoder/KiCad/RotaryEncoder/RotaryEncoder.kicad_pcb (KiCad board)
At the start: 2 copper layers, 39 x 39 mm, 15 parts, among them J1 Conn_01x06, U1 PEC11R-4325F-S0012

Commit message: Added hole description and dimensions
Other:
- board text added: "30mm"
- board text added: "M3"
Changed lines of the file:
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@@
+		(layer "B.SilkS")
+	)
+	(gr_line
+		(start 140.5 84.25)
+		(end 141 83.75)
+		(stroke
+			(width 0.2)
+			(type solid)
+		)
 		(layer "B.SilkS")
 	)
@@
 		)
 		(fill yes)
+		(layer "B.SilkS")
+	)
+	(gr_line
+		(start 140.5 76.25)
+		(end 141 76.75)
+		(stroke
+			(width 0.2)
+			(type solid)
+		)
 		(layer "B.SilkS")
 	)
@@
 		(layer "B.SilkS")
 	)
+	(gr_line
+		(start 140.5 82.75)
+		(end 140.5 84.25)
+		(stroke
+			(width 0.2)
+			(type solid)
+		)
+		(layer "B.SilkS")
+	)
 	(gr_poly
 		(pts
@@
 		)
 		(fill yes)
+		(layer "B.SilkS")
+	)
+	(gr_line
+		(start 131 70.64125)
+		(end 129.5 70.64125)
+		(stroke
+			(width 0.2)
+			(type solid)
+		)
+		(layer "B.SilkS")
+	)
+	(gr_line
+		(start 140.5 76.25)
+		(end 140 76.75)
+		(stroke
+			(width 0.2)
+			(type solid)
+		)
 		(layer "B.SilkS")
 	)
@@
 		)
 		(fill yes)
+		(layer "B.SilkS")
+	)
+	(gr_line
+		(start 137.5 70.64125)
+		(end 137 70.14125)
+		(stroke
+			(width 0.2)
+			(type solid)
+		)
+		(layer "B.SilkS")
+	)
+	(gr_line
+		(start 129.5 70.64125)
+		(end 130 71.14125)
+		(stroke
+			(width 0.2)
+			(type solid)
+		)
 		(layer "B.SilkS")
 	)
@@
 		(layer "B.SilkS")
 	)
+	(gr_line
+		(start 140.5 77.75)
+		(end 140.5 76.25)
+		(stroke
+			(width 0.2)
+			(type solid)
+		)
+		(layer "B.SilkS")
+	)
+	(gr_line
+		(start 136 70.64125)
+		(end 137.5 70.64125)
+		(stroke
+			(width 0.2)
+			(type solid)
+		)
+		(layer "B.SilkS")
+	)
 	(gr_poly
 		(pts
@@
 	)
 	(gr_line
+		(start 140.5 84.25)
+		(end 140 83.75)
+		(stroke
+			(width 0.2)
+			(type solid)
+		)
+		(layer "B.SilkS")
+	)
+	(gr_line
+		(start 137.5 70.64125)
+		(end 137 71.14125)
+		(stroke
+			(width 0.2)
+			(type solid)
+		)
+		(layer "B.SilkS")
+	)
+	(gr_line
+		(start 129.5 70.64125)
+		(end 130 70.14125)
+		(stroke
+			(width 0.2)
+			(type solid)
+		)
+		(layer "B.SilkS")
+	)
+	(gr_line
 		(start 141 66)
 		(end 110 66)
@@
 		)
 	)
+	(gr_text "M3"
+		(at 112 98.25 -0)
+		(layer "B.SilkS")
+		(effects
+			(font
+				(size 1.5 1.5)
+				(thickness 0.3)
+				(bold yes)
+			)
+			(justify left bottom mirror)
+		)
+	)
 	(gr_text "VCC"
 		(at 110 93.5 0)
@@
 		)
 	)
+	(gr_text "M3"
+		(at 142.25 74.75 -0)
+		(layer "B.SilkS")
+		(effects
+			(font
+				(size 1.5 1.5)
+				(thickness 0.3)
+				(bold yes)
+			)
+			(justify left bottom mirror)
+		)
+	)
+	(gr_text "M3"
+		(at 142.25 98.5 -0)
+		(layer "B.SilkS")
+		(effects
+			(font
+				(size 1.5 1.5)
+				(thickness 0.3)
+				(bold yes)
+			)
+			(justify left bottom mirror)
+		)
+	)
 	(gr_text "A"
 		(at 110 81 0)
@@
 		)
 	)
+	(gr_text "30mm"
+		(at 140 82.5 270)
+		(layer "B.SilkS")
+		(effects
+			(font
+				(size 1 1)
+				(thickness 0.125)
+			)
+			(justify left bottom mirror)
+		)
+	)
+	(gr_text "M3"
+		(at 112 74.75 -0)
+		(layer "B.SilkS")
+		(effects
+			(font
+				(size 1.5 1.5)
+				(thickness 0.3)
+				(bold yes)
+			)
+			(justify left bottom mirror)
+		)
+	)
 	(gr_text "GND"
 		(at 110 90.5 0)
@@
 	(gr_text "pmod.robotikabrno.cz/"
 		(at 138 102.5 0)
+		(layer "B.SilkS")
+		(effects
+			(font
+				(size 1 1)
+				(thickness 0.125)
+			)
+			(justify left bottom mirror)
+		)
+	)
+	(gr_text "30mm"
+		(at 135.75 71.14125 0)
 		(layer "B.SilkS")
 		(effects
@@
 		)
 	)
+	(group ""
+		(members "720184e0-9b3c-4cde-92df-0df7ea1846dd" "8531a072-f5ec-46dd-ac1f-e552872edddc"
+			"93b77d02-8b3c-4a19-9fb5-e7a65dabe338" "d05e4187-ff91-40c7-ae87-41dac3fb346b"
+			"e047e068-493a-45b1-a6d0-f2ba2d7a604d" "f616b6ce-b032-42dd-a3c7-a44c4917bf8d"
+			"ff52a18a-b10e-4cd6-88aa-77af623d83ff"
+		)
+	)
+	(group ""
+		(members "25680a20-e8ca-4667-985b-50a4e490737f" "51c1ba5f-dabb-459f-9575-1e07a2330a43"
+			"52507fe3-42f3-4e49-b25f-ff9090c0c760" "5ca7acc0-789d-48d9-b0f9-b3a400602163"
+			"733cd084-8c98-43ce-8c96-7efb26870849" "c9e9acb8-77f3-48aa-aadb-2151fb4af69e"
+			"dd4dfde3-0ca1-4344-aad9-b7e435ed5d5d"
+		)
+	)

Commit message: minor fixes
Routing:
- net GND: vias 0 -> 17
Changed lines of the file:
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@@
 			(psa4output no)
 			(plot_black_and_white yes)
+			(plotinvisibletext no)
 			(sketchpadsonfab no)
 			(plotpadnumbers no)
@@
 		(net 2)
 	)
+	(via
+		(at 141.6 80.2)
+		(size 0.6)
+		(drill 0.3)
+		(layers "F.Cu" "B.Cu")
+		(free yes)
+		(net 2)
+	)
+	(via
+		(at 142 92)
+		(size 0.6)
+		(drill 0.3)
+		(layers "F.Cu" "B.Cu")
+		(free yes)
+		(net 2)
+	)
+	(via
+		(at 119 68)
+		(size 0.6)
+		(drill 0.3)
+		(layers "F.Cu" "B.Cu")
+		(free yes)
+		(net 2)
+	)
+	(via
+		(at 129.8 92)
+		(size 0.6)
+		(drill 0.3)
+		(layers "F.Cu" "B.Cu")
+		(free yes)
+		(net 2)
+	)
+	(via
+		(at 120 87)
+		(size 0.6)
+		(drill 0.3)
+		(layers "F.Cu" "B.Cu")
+		(free yes)
+		(net 2)
+	)
+	(via
+		(at 130.8 78.6)
+		(size 0.6)
+		(drill 0.3)
+		(layers "F.Cu" "B.Cu")
+		(free yes)
+		(net 2)
+	)
+	(via
+		(at 108.4 81.2)
+		(size 0.6)
+		(drill 0.3)
+		(layers "F.Cu" "B.Cu")
+		(free yes)
+		(net 2)
+	)
+	(via
+		(at 132 67.8)
+		(size 0.6)
+		(drill 0.3)
+		(layers "F.Cu" "B.Cu")
+		(free yes)
+		(net 2)
+	)
+	(via
+		(at 136.4 88.2)
+		(size 0.6)
+		(drill 0.3)
+		(layers "F.Cu" "B.Cu")
+		(free yes)
+		(net 2)
+	)
+	(via
+		(at 114.4 76.6)
+		(size 0.6)
+		(drill 0.3)
+		(layers "F.Cu" "B.Cu")
+		(free yes)
+		(net 2)
+	)
+	(via
+		(at 132.6 100.8)
+		(size 0.6)
+		(drill 0.3)
+		(layers "F.Cu" "B.Cu")
+		(free yes)
+		(net 2)
+	)
+	(via
+		(at 127 76.2)
+		(size 0.6)
+		(drill 0.3)
+		(layers "F.Cu" "B.Cu")
+		(free yes)
+		(net 2)
+	)
+	(via
+		(at 128.4 84.2)
+		(size 0.6)
+		(drill 0.3)
+		(layers "F.Cu" "B.Cu")
+		(free yes)
+		(net 2)
+	)
+	(via
+		(at 123.2 86.8)
+		(size 0.6)
+		(drill 0.3)
+		(layers "F.Cu" "B.Cu")
+		(free yes)
+		(net 2)
+	)
+	(via
+		(at 127.4 89)
+		(size 0.6)
+		(drill 0.3)
+		(layers "F.Cu" "B.Cu")
+		(free yes)
+		(net 2)
+	)
+	(via
+		(at 120.4 102)
+		(size 0.6)
+		(drill 0.3)
+		(layers "F.Cu" "B.Cu")
+		(free yes)
+		(net 2)
+	)
+	(via
+		(at 108.4 91.4)
+		(size 0.6)
+		(drill 0.3)
+		(layers "F.Cu" "B.Cu")
+		(free yes)
+		(net 2)
+	)
