File: pmod/Temperature/KiCad/robocamp_temperature.kicad_pcb (KiCad board)
At the start: 2 copper layers, 23 x 17 mm, 3 parts, among them J1 Conn_01x06_Pin, U1 DS18B20

Commit message: Added link and logo
Other:
- board text added: "Temperature"
- board text added: "pmod.robotikabrno.cz/"

Commit message: rewrote link to match google sheets
Other:
- board text added: "thermometer"
- board text removed: "Temperature"
Changed lines of the file:
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@@
 		)
 	)
-	(gr_text "Temperature"
-		(at 148.75 107.75 -0)
+	(gr_text "thermometer"
+		(at 148.75 107.75 0)
 		(layer "B.SilkS")
 		(effects
