File: pmod/Microphone/KiCad/microphone.kicad_pcb (KiCad board)
At the start: 2 copper layers, 43.5 x 34 mm, 17 parts, among them J1 Conn_01x06_Pin, U1 LMV321, U2 LMV321

Commit message: Hyperlink to board
Parts:
- added H4: M3, MountingHole:MountingHole_3.2mm_M3, F.Cu at (141.0, 114.0)
- H1, H2, H3: value MountingHole -> M3
- moved J1 5.36 mm to (141.0, 95.3)
- moved H1 1.50 mm to (141.0, 88.0)
- moved H2 1.50 mm to (107.0, 88.0)
- moved H3 1.50 mm to (107.0, 114.0)
Routing:
- net +3V3: track 18.5 -> 46.7 mm
- net Net-(J1-Pin_6): track 33.7 -> 35.2 mm
Other:
- board text added: "MIC"
- board text added: "https://pmod.robotikabrno.cz/pmod/"
Changed lines of the file:
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@@
 	(footprint "MountingHole:MountingHole_3.2mm_M3"
 		(layer "F.Cu")
-		(at 141 89.5)
+		(at 141 88)
 		(descr "Mounting Hole 3.2mm, no annular, M3")
 		(tags "mounting hole 3.2mm no annular m3")
@@
 			(at 0 -4.2 0)
 			(layer "F.SilkS")
+			(hide yes)
 			(effects
 				(font
@@
 			)
 		)
-		(property "Value" "MountingHole"
+		(property "Value" "M3"
 			(at 0 4.2 0)
 			(layer "F.Fab")
@@
 	(footprint "MountingHole:MountingHole_3.2mm_M3"
 		(layer "F.Cu")
-		(at 107 112.5)
+		(at 107 114)
 		(descr "Mounting Hole 3.2mm, no annular, M3")
 		(tags "mounting hole 3.2mm no annular m3")
@@
 			(at 0 -4.2 0)
 			(layer "F.SilkS")
+			(hide yes)
 			(effects
 				(font
@@
 			)
 		)
-		(property "Value" "MountingHole"
-			(at 0 4.2 0)
+		(property "Value" "M3"
+			(at 0 -4 0)
 			(layer "F.Fab")
 			(effects
@@
 	(footprint "MountingHole:MountingHole_3.2mm_M3"
 		(layer "F.Cu")
-		(at 107 89.5)
+		(at 141 114)
+		(descr "Mounting Hole 3.2mm, no annular, M3")
+		(tags "mounting hole 3.2mm no annular m3")
+		(property "Reference" "H4"
+			(at 0 -4.2 0)
+			(layer "F.SilkS")
+			(hide yes)
+			(effects
+				(font
+					(size 1 1)
+					(thickness 0.15)
+				)
+			)
+		)
+		(property "Value" "M3"
+			(at 0 -4 0)
+			(layer "F.Fab")
+			(effects
+				(font
+					(size 1 1)
+					(thickness 0.15)
+				)
+			)
+		)
+		(property "Footprint" "MountingHole:MountingHole_3.2mm_M3"
+			(at 0 0 0)
+			(unlocked yes)
+			(layer "F.Fab")
+			(hide yes)
+			(effects
+				(font
+					(size 1.27 1.27)
+					(thickness 0.15)
+				)
+			)
+		)
+		(property "Datasheet" ""
+			(at 0 0 0)
+			(unlocked yes)
+			(layer "F.Fab")
+			(hide yes)
+			(effects
+				(font
+					(size 1.27 1.27)
+					(thickness 0.15)
+				)
+			)
+		)
+		(property "Description" "Mounting Hole without connection"
+			(at 0 0 0)
+			(unlocked yes)
+			(layer "F.Fab")
+			(hide yes)
+			(effects
+				(font
+					(size 1.27 1.27)
+					(thickness 0.15)
+				)
+			)
+		)
+		(property ki_fp_filters "MountingHole*")
+		(sheetname "Hlavní")
+		(sheetfile "microphone.kicad_sch")
+		(attr exclude_from_pos_files exclude_from_bom)
+		(fp_circle
+			(center 0 0)
+			(end 3.2 0)
+			(stroke
+				(width 0.15)
+				(type solid)
+			)
+			(fill none)
+			(layer "Cmts.User")
+		)
+		(fp_circle
+			(center 0 0)
+			(end 3.45 0)
+			(stroke
+				(width 0.05)
+				(type solid)
+			)
+			(fill none)
+			(layer "F.CrtYd")
+		)
+		(fp_text user "${REFERENCE}"
+			(at 0 0 0)
+			(layer "F.Fab")
+			(effects
+				(font
+					(size 1 1)
+					(thickness 0.15)
+				)
+			)
+		)
+		(pad "" np_thru_hole circle
+			(at 0 0)
+			(size 3.2 3.2)
+			(drill 3.2)
+			(layers "*.Cu" "*.Mask" "In1.Cu" "In2.Cu" "In3.Cu" "In4.Cu" "In5.Cu" "In6.Cu"
+				"In7.Cu" "In8.Cu" "In9.Cu" "In10.Cu" "In11.Cu" "In12.Cu" "In13.Cu" "In14.Cu"
+				"In15.Cu" "In16.Cu" "In17.Cu" "In18.Cu" "In19.Cu" "In20.Cu" "In21.Cu"
+				"In22.Cu" "In23.Cu" "In24.Cu" "In25.Cu" "In26.Cu" "In27.Cu" "In28.Cu"
+				"In29.Cu" "In30.Cu"
+			)
+		)
+	)
+	(footprint "MountingHole:MountingHole_3.2mm_M3"
+		(layer "F.Cu")
+		(at 107 88)
 		(descr "Mounting Hole 3.2mm, no annular, M3")
 		(tags "mounting hole 3.2mm no annular m3")
@@
 			(at 0 -4.2 0)
 			(layer "F.SilkS")
+			(hide yes)
 			(effects
 				(font
@@
 			)
 		)
-		(property "Value" "MountingHole"
+		(property "Value" "M3"
 			(at 0 4.2 0)
 			(layer "F.Fab")
@@
 		)
 		(property "Value" "CMEJ-9745-37-P"
-			(at 7.93 6.165 90)
+			(at 5.23 0 90)
 			(layer "F.Fab")
 			(effects
@@
 	(footprint "Connector_PinHeader_2.54mm:PinHeader_1x06_P2.54mm_Horizontal"
 		(layer "F.Cu")
-		(at 140.625 100.65)
+		(at 141 95.3)
 		(descr "Through hole angled pin header, 1x06, 2.54mm pitch, 6mm pin length, single row")
 		(tags "Through hole angled pin header THT 1x06 2.54mm single row")
@@
 		(layer "Edge.Cuts")
 	)
+	(gr_text "https://pmod.robotikabrno.cz/pmod/"
+		(at 104.14 116.84 90)
+		(layer "F.SilkS")
+		(effects
+			(font
+				(size 1 1)
+				(thickness 0.125)
+			)
+			(justify left bottom)
+		)
+	)
+	(gr_text "MIC"
+		(at 104.1654 88.392 90)
+		(layer "F.SilkS")
+		(effects
+			(font
+				(size 1 1)
+				(thickness 0.2)
+				(bold yes)
+			)
+			(justify left bottom)
+		)
+	)
 	(segment
 		(start 127 98)
@@
 	)
 	(segment
-		(start 140.625 100.65)
-		(end 140.35 100.65)
-		(width 0.2)
+		(start 139 97)
+		(end 140.7 95.3)
+		(width 0.5)
+		(layer "F.Cu")
+		(net 5)
+	)
+	(segment
+		(start 134.12 88.5)
+		(end 141 95.38)
+		(width 0.5)
+		(layer "F.Cu")
+		(net 5)
+	)
+	(segment
+		(start 140.7 95.3)
+		(end 141 95.3)
+		(width 0.5)
 		(layer "F.Cu")
 		(net 5)
@@
 	)
 	(segment
+		(start 139 111)
+		(end 139 97)
+		(width 0.5)
+		(layer "F.Cu")
+		(net 5)
+	)
+	(segment
+		(start 132.08 88.5)
+		(end 134.12 88.5)
+		(width 0.5)
+		(layer "F.Cu")
+		(net 5)
+	)
+	(segment
 		(start 126.05 91.95)
 		(end 126.05 94.8625)
@@
 	)
 	(segment
-		(start 131.5 112)
-		(end 137 112)
-		(width 0.5)
-		(layer "B.Cu")
-		(net 7)
-	)
-	(segment
-		(start 138.35 113.35)
-		(end 140.625 113.35)
+		(start 131 101.5)
+		(end 131 95)
 		(width 0.5)
 		(layer "B.Cu")
@@
 	(segment
 		(start 137 112)
-		(end 138.35 113.35)
+		(end 141 108)
 		(width 0.5)
 		(layer "B.Cu")
@@
 	)
 	(segment
-		(start 131 101.5)
-		(end 131 95)
+		(start 131.5 112)
+		(end 137 112)
 		(width 0.5)
 		(layer "B.Cu")
@@
 	)
 	(segment
+		(start 140.625 100.65)
+		(end 140.35 100.65)
+		(width 0.2)
+		(layer "F.Cu")
+		(net 9)
+	)
+	(segment

Commit message: minor fixes
Parts:
- removed U2: LMV321, Package_TO_SOT_SMD:SOT-353_SC-70-5_Handsoldering
- C1: value 0.1u -> 0.2u
- R1, R2: value 2k -> 1k
Routing:
- net GND: track 2.96 -> 0.69 mm

Commit message: fix: small pcb fixes
Parts:
- moved J1 0.58 mm to (141.5, 95.1)
Routing:
- net +3V3: track 46.7 -> 47.5 mm
- net Net-(J1-Pin_6): track 35.2 -> 35.8 mm
Other:
- board text added: "pmod.robotikabrno.cz/"
- board text removed: "https://pmod.robotikabrno.cz/pmod/"
Changed lines of the file:
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@@
 			(psa4output no)
 			(plot_black_and_white yes)
-			(plotinvisibletext no)
 			(sketchpadsonfab no)
 			(plotpadnumbers no)
@@
 		)
 		(property "Value" "1uF"
-			(at 2.5 2.2 90)
+			(at -2.448 -0.025 90)
 			(layer "F.Fab")
 			(effects
@@
 	(footprint "Connector_PinHeader_2.54mm:PinHeader_1x06_P2.54mm_Horizontal"
 		(layer "F.Cu")
-		(at 141 95.3)
+		(at 141.548 95.123)
 		(descr "Through hole angled pin header, 1x06, 2.54mm pitch, 6mm pin length, single row")
 		(tags "Through hole angled pin header THT 1x06 2.54mm single row")
@@
 		)
 		(property "Value" "10k"
-			(at 5.08 2.37 90)
+			(at 7.488 0 90)
 			(layer "F.Fab")
 			(effects
@@
 		(layer "Edge.Cuts")
 	)
-	(gr_text "https://pmod.robotikabrno.cz/pmod/"
-		(at 104.14 116.84 90)
+	(gr_text "pmod.robotikabrno.cz/"
+		(at 104.648 111.252 90)
 		(layer "F.SilkS")
 		(effects
@@
 	)
 	(gr_text "MIC"
-		(at 104.1654 88.392 90)
+		(at 104.902 94.234 90)
 		(layer "F.SilkS")
 		(effects
@@
 	)
 	(segment
-		(start 139 97)
-		(end 140.7 95.3)
+		(start 132.08 88.5)
+		(end 133.712 88.5)
 		(width 0.5)
 		(layer "F.Cu")
@@
 	)
 	(segment
-		(start 134.12 88.5)
-		(end 141 95.38)
+		(start 133.712 88.5)
+		(end 140.335 95.123)
 		(width 0.5)
 		(layer "F.Cu")
@@
 	)
 	(segment
-		(start 140.7 95.3)
-		(end 141 95.3)
+		(start 129.5 88.5)
+		(end 132.08 88.5)
 		(width 0.5)
 		(layer "F.Cu")
@@
 	)
 	(segment
-		(start 129.5 88.5)
-		(end 132.08 88.5)
+		(start 132.58 114.5)
+		(end 135.5 114.5)
 		(width 0.5)
 		(layer "F.Cu")
@@
 	)
 	(segment
-		(start 135.5 114.5)
-		(end 139 111)
+		(start 141.548 95.123)
+		(end 141.371 95.3)
 		(width 0.5)
 		(layer "F.Cu")
@@
 	)
 	(segment
-		(start 139 111)
-		(end 139 97)
+		(start 126.05 91.95)
+		(end 126.05 94.8625)
 		(width 0.5)
 		(layer "F.Cu")
@@
 	)
 	(segment
-		(start 132.08 88.5)
-		(end 134.12 88.5)
+		(start 139 96.458)
+		(end 140.335 95.123)
 		(width 0.5)
 		(layer "F.Cu")
@@
 	)
 	(segment
-		(start 126.05 91.95)
-		(end 126.05 94.8625)
+		(start 141.371 95.3)
+		(end 141 95.3)
+		(width 0.5)
+		(layer "F.Cu")
+		(net 5)
+	)
+	(segment
+		(start 135.5 114.5)
+		(end 139 111)
+		(width 0.5)
+		(layer "F.Cu")
+		(net 5)
+	)
+	(segment
+		(start 139 111)
+		(end 139 96.458)
 		(width 0.5)
 		(layer "F.Cu")
@@
 	)
 	(segment
-		(start 132.58 114.5)
-		(end 135.5 114.5)
+		(start 140.335 95.123)
+		(end 141.548 95.123)
 		(width 0.5)
 		(layer "F.Cu")
@@
 	)
 	(segment
+		(start 141.177 107.823)
+		(end 141.548 107.823)
+		(width 0.5)
+		(layer "B.Cu")
+		(net 7)
+	)
+	(segment
 		(start 131 101.5)
 		(end 131 95)
@@
 	)
 	(segment
-		(start 137 112)
-		(end 141 108)
+		(start 129 109.5)
+		(end 131.5 112)
 		(width 0.5)
 		(layer "B.Cu")
@@
 	)
 	(segment
-		(start 126.5 106)
-		(end 131 101.5)
+		(start 137 112)
+		(end 141.177 107.823)
 		(width 0.5)
 		(layer "B.Cu")
@@
 	)
 	(segment
-		(start 129 109.5)
-		(end 131.5 112)
+		(start 126.5 106)
+		(end 131 101.5)
 		(width 0.5)
 		(layer "B.Cu")
@@
 	)
 	(segment
-		(start 140.625 100.65)
-		(end 140.35 100.65)
-		(width 0.2)
-		(layer "F.Cu")
-		(net 9)
-	)
-	(segment
