File: pmod/RotaryEncoder/KiCad/RotaryEncoder.kicad_pcb (KiCad board)
At the start: 2 copper layers, 39 x 39 mm, 15 parts, among them J1 Conn_01x06, U1 PEC11R-4325F-S0012

Commit message: fix: small pcb fixes
Changed lines of the file:
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@@
 			(psa4output no)
 			(plot_black_and_white yes)
-			(plotinvisibletext no)
 			(sketchpadsonfab no)
 			(plotpadnumbers no)
@@
 			)
 		)
-		(pad "1" thru_hole circle
+		(pad "1" thru_hole oval
 			(at 0 14.5 90)
-			(size 1.5 1.5)
+			(size 1.6 2)
 			(drill 1)
 			(layers "*.Cu" "*.Mask")
@@
 			(pintype "passive")
 		)
-		(pad "2" thru_hole circle
+		(pad "2" thru_hole oval
 			(at 5 14.5 90)
-			(size 1.5 1.5)
+			(size 1.6 2)
 			(drill 1)
 			(layers "*.Cu" "*.Mask")
@@
 		(pad "A1" thru_hole rect
 			(at 0 0 90)
-			(size 1.5 1.5)
+			(size 1.6 2)
 			(drill 1)
 			(layers "*.Cu" "*.Mask")
@@
 			(pintype "passive")
 		)
-		(pad "B1" thru_hole circle
+		(pad "B1" thru_hole oval
 			(at 5 0 90)
-			(size 1.5 1.5)
+			(size 1.6 2)
 			(drill 1)
 			(layers "*.Cu" "*.Mask")
@@
 			(pintype "passive")
 		)
-		(pad "C1" thru_hole circle
+		(pad "C1" thru_hole oval
 			(at 2.5 0 90)
-			(size 1.5 1.5)
+			(size 1.6 2)
 			(drill 1)
 			(layers "*.Cu" "*.Mask")
@@
 			(font
 				(size 1 1)
-				(thickness 0.1)
+				(thickness 0.125)
 			)
 			(justify left bottom mirror)
@@
 			(font
 				(size 1 1)
-				(thickness 0.1)
+				(thickness 0.125)
 			)
 			(justify left bottom mirror)
@@
 			(font
 				(size 1 1)
-				(thickness 0.1)
+				(thickness 0.125)
 			)
 			(justify left bottom mirror)
@@
 			(font
 				(size 1 1)
-				(thickness 0.1)
+				(thickness 0.125)
 			)
 			(justify left mirror)
@@
 			(font
 				(size 1 1)
-				(thickness 0.1)
+				(thickness 0.125)
 			)
 			(justify left bottom mirror)
