File: pmod/prototyp/KiCad/prototyp.kicad_sch (KiCad schematic)
At the start: 113 parts, among them J1 Conn_01x06_Pin

Commit message: fix: prepare all board for manufacturing
Parts:
- added H113, H114: MountingHole, MountingHole:MountingHole_3.2mm_M3, symbol Mechanical:MountingHole
- H1, H10, H100, H101, H102, H103, H104, H105, H106, H107, H108, H109, H11, H110, H111, H112, H12, H13, H14, H15, H16, H17, H18, H19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: value ~ -> (none)
Connections:
- no-connect marks 1 -> 0
