File: pmod/photoresistor/KiCad/photoresistor.kicad_pcb (KiCad board)
At the start: 2 copper layers, 20 x 16 mm, 4 parts, among them J2 Conn_01x06_Pin

Commit message: docs: add images, fix docs
Routing:
- net GND: vias 8 -> 7
Changed lines of the file:
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@@
-	)
-	(via
-		(at 129.5 108.5)
-		(size 0.6)
-		(drill 0.3)
-		(layers "F.Cu" "B.Cu")
-		(free yes)
-		(net "GND")
 	)
 	(via
