File: DPad/KiCad/dpad.kicad_sch (KiCad schematic)
At the start: 13 parts, among them SW1 SW_Push, SW2 SW_Push, SW3 SW_Push, SW4 SW_Push

Commit message: Deployed 7db42b7 with MkDocs version: 1.6.0
Parts:
- added C1, C2, C3, C4: 1uF, Custom:C_Disc_D6.0mm_W4mm_P5.00mm, symbol Device:C
- PMOD1: footprint Connector_PinHeader_2.54mm:PinHeader_1x06_P2.54mm_Vertical -> Connector_PinHeader_2.54mm:PinHeader_1x06_P2.54mm_Horizontal
- SW1, SW2, SW3, SW4: footprint Button_Switch_THT:SW_PUSH-12mm_Wuerth-430476085716 -> Custom:SW_PUSH-12mm
Connections:
- net GND: now also C1.1, C2.1, C3.1, C4.1
- net IO1: now also C1.2
- net IO2: now also C2.2
- net IO3: now also C3.2
- net IO4: now also C4.2
Other:
- moved on the sheet: R1, R2, R3, R4, SW1, SW2, SW3, SW4

Commit message: Deployed d972a79 with MkDocs version: 1.6.0
Other:
- moved on the sheet: C1, C2, C3, C4, H1, H2, H3, H4, PMOD1, R1, R2, R3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
