File: IR/KiCad/IR.kicad_sch (KiCad schematic)
At the start: 4 parts, among them J1 Conn_01x06

Commit message: Deployed de0c2bf with MkDocs version: 1.6.0
Parts:
- D1: value SFH4550 -> IR
- R1: value 180 -> 100
Connections:
- no-connect marks 0 -> 1
Changed lines of the file:
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@@
 	(generator_version "9.0")
 	(paper "A4")
+	(no_connect
+		(at 88.9 73.66)
+	)
 	(wire
 		(pts
@@
 			)
 		)
-		(property "Value" "SFH4550"
+		(property "Value" "IR"
 			(at 114.3 76.0729 90)
 			(effects
@@
 			)
 		)
-		(property "Value" "180"
+		(property "Value" "100"
 			(at 114.3 83.312 0)
 			(effects
