File: RFID/KiCad/RFID.kicad_sch (KiCad schematic)
At the start: 5 parts, among them J1 SPI IN, J2 RFID-RC522, J3 SPI OUT, J4 RST

Commit message: Deployed d972a79 with MkDocs version: 1.6.0
Connections:
- net +3.3V: now also J3.1 (Pin_1); no longer J3.6 (Pin_6)
- net GND: now also J3.2 (Pin_2); no longer J3.5 (Pin_5)
- net MISO: now also J3.4 (Pin_4); no longer J3.3 (Pin_3)
- net MOSI: now also J3.5 (Pin_5); no longer J3.2 (Pin_2)
- net SCK: now also J3.3 (Pin_3); no longer J3.4 (Pin_4)
- net SS: now also J3.6 (Pin_6); no longer J3.1 (Pin_1)
