File: r-encoder/KiCad/RotaryEncoder.kicad_sch (KiCad schematic)
At the start: 15 parts, among them J1 Conn_01x06, U1 PEC11R-4325F-S0012

Commit message: Deployed d972a79 with MkDocs version: 1.6.0
Parts:
- C1, C2, C3: value 0.01uF -> 10nF
Connections:
- net A: now also J1.3 (Pin_3); no longer J1.4 (Pin_4)
- net B: now also J1.4 (Pin_4); no longer J1.3 (Pin_3)
- net BTN: now also J1.5 (Pin_5); no longer J1.2 (Pin_2)
- net GND: now also J1.2 (Pin_2); no longer J1.5 (Pin_5)
- net VCC: now also J1.1 (Pin_1); no longer J1.6 (Pin_6)
Other:
- moved on the sheet: C1, C2, C3, H1, H2, H3, H4, R1, R2, R3, R4, R5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
