File: motor-driver/KiCad/pmod-motordriver.kicad_pcb (KiCad board)
At the start: 2 copper layers, 38.2 x 16.2 mm, 14 parts, among them J1 Conn_01x06_Pin, J2 Screw_Terminal_01x02, J3 Screw_Terminal_01x02, J4 Screw_Terminal_01x02, Q1 AO3401A, U1 DRV8833PWP

Commit message: Deployed 05c467d with MkDocs version: 1.6.0
Changed lines of the file:
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@@
 			(psa4output no)
 			(plot_black_and_white yes)
+			(plotinvisibletext no)
 			(sketchpadsonfab no)
 			(plotpadnumbers no)
@@
 	)
 	(segment
-		(start 175.08 105.75)
-		(end 174.58 106.25)
+		(start 182.95 106.2)
+		(end 174.63 106.2)
 		(width 0.8)
 		(layer "F.Cu")
@@
 	)
 	(segment
-		(start 182.5 105.75)
-		(end 175.08 105.75)
-		(width 0.8)
+		(start 156.85 117)
+		(end 156.5 117)
+		(width 0.2)
 		(layer "F.Cu")
 		(net 16)
@@
 	(segment
 		(start 183 106.25)
-		(end 182.5 105.75)
+		(end 182.95 106.2)
 		(width 0.8)
 		(layer "F.Cu")
@@
 	)
 	(segment
-		(start 156.85 117)
-		(end 156.5 117)
-		(width 0.2)
-		(layer "F.Cu")
-		(net 16)
-	)
-	(segment
 		(start 156.5 117)
 		(end 155.75 116.25)
@@
 		(net 16)
 	)
+	(segment
+		(start 174.63 106.2)
+		(end 174.58 106.25)
+		(width 0.8)
+		(layer "F.Cu")
+		(net 16)
+	)
 	(via
 		(at 155.75 116.25)
@@
 		(polygon
 			(pts
-				(xy 179 108.5) (xy 179.75 107.75) (xy 181.75 107.75) (xy 181.75 106.25) (xy 175.75 106.25) (xy 175.75 106.5)
+				(xy 179 108.5) (xy 179.2 108.4) (xy 179.55 108.4) (xy 179.55 106.25) (xy 175.75 106.25) (xy 175.75 106.5)
 				(xy 175 107.25) (xy 174.25 107.25) (xy 173.5 106.5) (xy 173.5 105.5) (xy 173.25 105.25) (xy 171 105.25)
 				(xy 170.75 105.5) (xy 170.75 107.25) (xy 174 109.25) (xy 177.25 109.25) (xy 177.25 108.75) (xy 177.5 108.5)

Commit message: Deployed d972a79 with MkDocs version: 1.6.0
Parts:
- removed J3: Screw_Terminal_01x02, TerminalBlock_TE-Connectivity:TerminalBlock_TE_282834-2_1x02_P2.54mm_Horizontal
- added H1: MountingHole, MountingHole:MountingHole_3.2mm_M3, F.Cu at (176.5, 101.5)
- added J5: Screw_Terminal_01x04, TerminalBlock_Phoenix:TerminalBlock_Phoenix_MKDS-1,5-4-5.08_1x04_P5.08mm_Horizontal, F.Cu at (194.7, 116.1)
- J2: footprint TerminalBlock_TE-Connectivity:TerminalBlock_TE_282834-2_1x02_P2.54mm_Horizontal -> TerminalBlock_Phoenix:TerminalBlock_Phoenix_MKDS-1,5-2-5.08_1x02_P5.08mm_Horizontal
- J4: value Screw_Terminal_01x02 -> Conn_01x04_Pin; footprint TerminalBlock_TE-Connectivity:TerminalBlock_TE_282834-2_1x02_P2.54mm_Horizontal -> Connector_PinHeader_2.54mm:PinHeader_1x04_P2.54mm_Vertical
- R2: value 470 -> 1k
- moved J4 36.6 mm to (187.0, 112.3), turned to 180 degrees
- moved R2 29.3 mm to (182.5, 101.5), turned to 90 degrees
- moved D1 27.5 mm to (181.5, 99.0), turned to 0 degrees
- moved J1 26.1 mm to (158.4, 114.8), turned to 180 degrees
- moved J2 19.6 mm to (177.0, 117.0), turned to 0 degrees
- moved Q1 16.5 mm to (162.8, 112.5), turned to -90 degrees
- moved C2 11.7 mm to (165.2, 108.5), turned to -90 degrees
- moved R1 10.6 mm to (172.0, 113.5), turned to 0 degrees
- moved JP1 10.5 mm to (171.5, 116.5), turned to -90 degrees
- moved U1 9.98 mm to (175.5, 108.5), turned to 180 degrees
- moved C4 8.08 mm to (169.2, 106.8), turned to -90 degrees
- moved C1 8.04 mm to (167.2, 108.5), turned to -90 degrees
- moved C3 3.64 mm to (169.0, 111.0), turned to 180 degrees
- renumbered C9 to C2, C2 to C3, C3 to C4
Connections:
- J4 pad 1: Net-(J4-Pin_1) -> /AOUT1
- J4 pad 2: Net-(J4-Pin_2) -> /AOUT2
- U1 pad 2: Net-(J3-Pin_1) -> /AOUT1
- U1 pad 4: Net-(J3-Pin_2) -> /AOUT2
- U1 pad 5: Net-(J4-Pin_1) -> /BOUT2
- U1 pad 7: Net-(J4-Pin_2) -> /BOUT1
Routing:
- net Net-(J3-Pin_1): track 14.3 -> 0.00 mm
- net Net-(J4-Pin_2): track 14.3 -> 0.00 mm
- net Net-(J3-Pin_2): track 14.0 -> 0.00 mm
- net Net-(J4-Pin_1): track 14.0 -> 0.00 mm
- net Net-(J2-Pin_1): track 11.2 -> 0.00 mm
- net VCC: track 13.6 -> 3.66 mm
- net /BOUT1: track 0.00 -> 9.25 mm
- net /AOUT1: track 0.00 -> 9.25 mm
- net /BOUT2: track 0.00 -> 8.20 mm
- net /AOUT2: track 0.00 -> 8.20 mm
- net Net-(JP1-C): track 7.41 -> 0.00 mm
- net +5V: track 44.4 -> 37.4 mm
- net GND: track 9.04 -> 3.66 mm, vias 15 -> 29
- net Net-(D1-K): track 3.63 -> 8.20 mm
- net Net-(U1-~{SLEEP}): track 4.68 -> 6.88 mm, vias 0 -> 2
- added copper zone on F.Cu, net /AOUT1
- added copper zone on F.Cu, net /AOUT2
- added copper zone on F.Cu, net /BOUT1
- added copper zone on F.Cu, net /BOUT2
- added copper zone on F.Cu, net Net-(J2-Pin_1)
Other:
- board size 38.2 x 16.2 mm -> 45 x 22 mm
- board text added: "+ A -"
- board text added: "- B +"
- board text added: "- EXT. +"
- board text added: "22mm"
- board text added: "45mm"
- board text added: "AIN1 AIN2 BIN1 BIN2 GND 5V"
- board text added: "motor-driver"
- board text added: "pmod.robotikabrno.cz/"
- board text removed: "+ MOTOR B -"
- board text removed: "- EXTERNAL +"
- board text removed: "- MOTOR A +"
- board text removed: "5V GND BIN2 BIN1 AIN2 AIN1"

Commit message: Deployed a122263 with MkDocs version: 1.6.0
Other:
- board text added: "A+"
- board text added: "B+"
- board text added: "GND"
Changed lines of the file:
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@@
 			(at 14.12 -6.32 90)
 			(layer "F.SilkS")
+			(hide yes)
 			(effects
 				(font
@@
 			(at 0 -2.38 0)
 			(layer "F.SilkS")
+			(hide yes)
 			(effects
 				(font
@@
 			(at 5.545 -6.32 0)
 			(layer "F.SilkS")
+			(hide yes)
 			(effects
 				(font
@@
 		(layer "Edge.Cuts")
 	)
+	(gr_text "B+"
+		(at 187.5 101 90)
+		(layer "F.SilkS")
+		(effects
+			(font
+				(size 1 1)
+				(bold yes)
+			)
+		)
+	)
+	(gr_text "A+"
+		(at 187.5 116.5 90)
+		(layer "F.SilkS")
+		(effects
+			(font
+				(size 1 1)
+				(bold yes)
+			)
+		)
+	)
 	(gr_text "FAULT"
 		(at 185.5 99 0)
@@
 		)
 	)
+	(gr_text "GND"
+		(at 182 110 0)
+		(layer "F.SilkS")
+		(effects
+			(font
+				(size 1.4 1.4)
+				(thickness 0.32)
+				(bold yes)
+			)
+		)
+	)
