File: prototyp/KiCad/prototyp.kicad_pcb (KiCad board)
At the start: 2 copper layers, 62 x 20 mm, 115 parts, among them J1 Conn_01x06_Pin

Commit message: Deployed a122263 with MkDocs version: 1.6.0
Changed lines of the file:
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@@
 			(at 2.185 -2.27 0)
 			(layer "F.SilkS")
+			(hide yes)
 			(effects
 				(font
