File: PIEZO/KiCad/PIEZO.kicad_pcb (KiCad board)
At the start: 2 copper layers, 37 x 32 mm, 8 parts, among them J1 Conn_01x06_Pin

Commit message: Deployed 77a73f4 with MkDocs version: 1.6.0
Parts:
- BZ1: value AZ-1740E-2P -> Buzzer; footprint Samacsys:AZ-1740E-2P -> PIEZO:buzzer
- moved G*** 5.50 mm to (89.0, 73.0)
- turned BZ1 to 0 degrees
Connections:
- BZ1 pad 1: GND -> Net-(BZ1-+)
- BZ1 pad 2: Net-(BZ1-Pad2) -> GND
- R1 pad 2: Net-(BZ1-Pad2) -> Net-(BZ1-+)
Routing:
- net Net-(BZ1-Pad2): track 12.5 -> 0.00 mm
- net Net-(BZ1-+): track 0.00 -> 12.5 mm
Other:
- board text added: "Buzzer"

Commit message: Deployed d972a79 with MkDocs version: 1.6.0
Parts:
- removed G***: LOGO, LOGO
- moved REF** 1.58 mm to (110.0, 75.0)
- moved REF** 1.58 mm to (110.0, 51.0)
- moved REF** 0.71 mm to (82.0, 75.0)
- moved REF** 0.71 mm to (82.0, 51.0)
- moved J1 0.23 mm to (81.9, 69.3)
Other:
- board size 37 x 32 mm -> 36 x 32 mm
- board text added: "32mm"
- board text added: "36mm"
- board text removed: "25mm"
- board text removed: "30mm"
- board text removed: "M3"
- board text removed: "Pmod Gadgets"

Commit message: Deployed 33ea02e with MkDocs version: 1.6.0
Parts:
- moved REF** 4.00 mm to (106.0, 75.0)
- moved REF** 4.00 mm to (106.0, 51.0)
Routing:
- net Net-(BZ1-+): track 12.5 -> 13.6 mm
Other:
- board size 36 x 32 mm -> 32 x 32 mm
- board text removed: "36mm"
- board text removed: "Buzzer"
