File: PIEZO/KiCad/PIEZO.kicad_sch (KiCad schematic)
At the start: 3 parts, among them J1 Conn_01x06_Pin

Commit message: Deployed 77a73f4 with MkDocs version: 1.6.0
Parts:
- removed BZ1: AZ-1740E-2P, Samacsys:AZ-1740E-2P, symbol buzzer:AZ-1720E-P-LF
- added BZ1: Buzzer, PIEZO:buzzer, symbol Device:Buzzer
Connections:
- net GND: now also BZ1.2 (-)
- net at R1.2: now also BZ1.1 (+)
Other:
- moved on the sheet: R1
Changed lines of the file:
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@@
 	(wire
 		(pts
-			(xy 199.39 97.79) (xy 198.12 97.79)
+			(xy 199.39 96.52) (xy 198.12 96.52)
 		)
 		(stroke
@@
 	(wire
 		(pts
-			(xy 198.12 100.33) (xy 207.01 100.33)
+			(xy 198.12 101.6) (xy 207.01 101.6)
 		)
 		(stroke
@@
 	(global_label "PWM"
 		(shape input)
-		(at 198.12 97.79 180)
+		(at 198.12 96.52 180)
 		(fields_autoplaced yes)
 		(effects
@@
 		)
 		(property "Intersheetrefs" "${INTERSHEET_REFS}"
-			(at 190.962 97.79 0)
+			(at 190.962 96.52 0)
 			(effects
 				(font
@@
 	(global_label "GND"
 		(shape input)
-		(at 198.12 100.33 180)
+		(at 198.12 101.6 180)
 		(fields_autoplaced yes)
 		(effects
@@
 		)
 		(property "Intersheetrefs" "${INTERSHEET_REFS}"
-			(at 191.2643 100.33 0)
+			(at 191.2643 101.6 0)
 			(effects
 				(font
@@
 	)
 	(symbol
-		(lib_id "buzzer:AZ-1720E-P-LF")
-		(at 207.01 97.79 0)
+		(lib_id "Device:Buzzer")
+		(at 209.55 99.06 0)
 		(unit 1)
 		(exclude_from_sim no)
@@
 		(fields_autoplaced yes)
 		(property "Reference" "BZ1"
-			(at 218.44 97.7899 0)
-			(effects
-				(font
-					(size 1.27 1.27)
-				)
-				(justify left)
-			)
-		)
-		(property "Value" "AZ-1740E-2P"
-			(at 218.44 100.3299 0)
-			(effects
-				(font
-					(size 1.27 1.27)
-				)
-				(justify left)
-			)
-		)
-		(property "Footprint" "Samacsys:AZ-1740E-2P"
-			(at 218.44 200.33 0)
-			(effects
-				(font
-					(size 1.27 1.27)
-				)
-				(justify left top)
-				(hide yes)
-			)
-		)
-		(property "Datasheet" "https://www.mouser.com/datasheet/2/1005/2020050867529-2325031.pdf"
-			(at 218.44 300.33 0)
-			(effects
-				(font
-					(size 1.27 1.27)
-				)
-				(justify left top)
-				(hide yes)
-			)
-		)
-		(property "Description" "Piezo Buzzers & Audio Indicators Piezo Buzzer 4000Hz 5VAC, 80dBA"
-			(at 207.01 97.79 0)
-			(effects
-				(font
-					(size 1.27 1.27)
-				)
-				(hide yes)
-			)
-		)
-		(property "Height" "7.8"
-			(at 218.44 500.33 0)
-			(effects
-				(font
-					(size 1.27 1.27)
-				)
-				(justify left top)
-				(hide yes)
-			)
-		)
-		(property "Manufacturer_Name" "AATC"
-			(at 218.44 600.33 0)
-			(effects
-				(font
-					(size 1.27 1.27)
-				)
-				(justify left top)
-				(hide yes)
-			)
-		)
-		(property "Manufacturer_Part_Number" "AZ-1720E-P-LF"
-			(at 218.44 700.33 0)
-			(effects
-				(font
-					(size 1.27 1.27)
-				)
-				(justify left top)
-				(hide yes)
-			)
-		)
-		(property "Mouser Part Number" ""
-			(at 218.44 800.33 0)
-			(effects
-				(font
-					(size 1.27 1.27)
-				)
-				(justify left top)
-				(hide yes)
-			)
-		)
-		(property "Mouser Price/Stock" ""
-			(at 218.44 900.33 0)
-			(effects
-				(font
-					(size 1.27 1.27)
-				)
-				(justify left top)
-				(hide yes)
-			)
-		)
-		(property "Arrow Part Number" ""
-			(at 218.44 1000.33 0)
-			(effects
-				(font
-					(size 1.27 1.27)
-				)
-				(justify left top)
-				(hide yes)
-			)
-		)
-		(property "Arrow Price/Stock" ""
-			(at 218.44 1100.33 0)
-			(effects
-				(font
-					(size 1.27 1.27)
-				)
-				(justify left top)
+			(at 213.36 97.7899 0)
+			(effects
+				(font
+					(size 1.27 1.27)
+				)
+				(justify left)
+			)
+		)
+		(property "Value" "Buzzer"
+			(at 213.36 100.3299 0)
+			(effects
+				(font
+					(size 1.27 1.27)
+				)
+				(justify left)
+			)
+		)
+		(property "Footprint" "PIEZO:buzzer"
+			(at 208.915 96.52 90)
+			(effects
+				(font
+					(size 1.27 1.27)
+				)
+				(hide yes)
+			)
+		)
+		(property "Datasheet" "~"
+			(at 208.915 96.52 90)
+			(effects
+				(font
+					(size 1.27 1.27)
+				)
+				(hide yes)
+			)
+		)
+		(property "Description" "Buzzer, polarized"
+			(at 209.55 99.06 0)
+			(effects
+				(font
+					(size 1.27 1.27)
+				)
 				(hide yes)
 			)
@@
 	(symbol
 		(lib_id "Device:R")
-		(at 203.2 97.79 90)
+		(at 203.2 96.52 90)
 		(unit 1)
 		(exclude_from_sim no)
@@
 		(fields_autoplaced yes)
 		(property "Reference" "R1"
-			(at 203.2 91.44 90)
+			(at 203.2 90.17 90)
 			(effects
 				(font
@@
 		)
 		(property "Value" "330R"
-			(at 203.2 93.98 90)
+			(at 203.2 92.71 90)
 			(effects
 				(font
@@
 		)
 		(property "Footprint" "Resistor_THT:R_Axial_DIN0207_L6.3mm_D2.5mm_P10.16mm_Horizontal"
-			(at 203.2 99.568 90)
+			(at 203.2 98.298 90)
 			(effects
 				(font
@@
 		)
 		(property "Datasheet" "~"
-			(at 203.2 97.79 0)
+			(at 203.2 96.52 0)
 			(effects
 				(font
@@
 		)
 		(property "Description" "Resistor"
-			(at 203.2 97.79 0)
-			(effects
-				(font
+			(at 203.2 96.52 0)
+			(effects
+				(font

Commit message: Deployed d972a79 with MkDocs version: 1.6.0
Connections:
- no-connect marks 0 -> 4
Changed lines of the file:
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@@
 (kicad_sch
-	(version 20250114)
+	(version 20260306)
 	(generator "eeschema")
-	(generator_version "9.0")
+	(generator_version "10.0")
 	(paper "A4")
+	(no_connect
+		(at 180.34 90.17)
+	)
+	(no_connect
+		(at 180.34 92.71)
+	)
+	(no_connect
+		(at 180.34 102.87)
+	)
+	(no_connect
+		(at 180.34 95.25)
+	)
 	(wire
 		(pts
@@
 		(property "Intersheetrefs" "${INTERSHEET_REFS}"
 			(at 187.498 97.79 0)
+			(hide yes)
+			(show_name no)
+			(do_not_autoplace no)
 			(effects
 				(font
@@
 				)
 				(justify left)
-				(hide yes)
 			)
 		)
@@
 		(property "Intersheetrefs" "${INTERSHEET_REFS}"
 			(at 190.962 96.52 0)
+			(hide yes)
+			(show_name no)
+			(do_not_autoplace no)
 			(effects
 				(font
@@
 				)
 				(justify right)
-				(hide yes)
 			)
 		)
@@
 		(property "Intersheetrefs" "${INTERSHEET_REFS}"
 			(at 191.2643 101.6 0)
+			(hide yes)
+			(show_name no)
+			(do_not_autoplace no)
 			(effects
 				(font
@@
 				)
 				(justify right)
-				(hide yes)
 			)
 		)
@@
 		(property "Intersheetrefs" "${INTERSHEET_REFS}"
 			(at 187.1957 100.33 0)
+			(hide yes)
+			(show_name no)
+			(do_not_autoplace no)
 			(effects
 				(font
@@
 				)
 				(justify left)
-				(hide yes)
 			)
 		)
@@
 		(mirror x)
 		(unit 1)
+		(body_style 1)
 		(exclude_from_sim no)
 		(in_bom yes)
 		(on_board yes)
+		(in_pos_files yes)
 		(dnp no)
 		(property "Reference" "J1"
 			(at 173.99 95.2499 0)
+			(show_name no)
+			(do_not_autoplace no)
 			(effects
 				(font
@@
 		(property "Value" "Conn_01x06_Pin"
 			(at 173.99 97.7899 0)
+			(show_name no)
+			(do_not_autoplace no)
 			(effects
 				(font
@@
 		(property "Footprint" "Connector_PinHeader_2.54mm:PinHeader_1x06_P2.54mm_Horizontal"
 			(at 175.26 97.79 0)
-			(effects
-				(font
-					(size 1.27 1.27)
-				)
-				(hide yes)
-			)
-		)
-		(property "Datasheet" "~"
+			(hide yes)
+			(show_name no)
+			(do_not_autoplace no)
+			(effects
+				(font
+					(size 1.27 1.27)
+				)
+			)
+		)
+		(property "Datasheet" ""
 			(at 175.26 97.79 0)
-			(effects
-				(font
-					(size 1.27 1.27)
-				)
-				(hide yes)
+			(hide yes)
+			(show_name no)
+			(do_not_autoplace no)
+			(effects
+				(font
+					(size 1.27 1.27)
+				)
 			)
 		)
 		(property "Description" "Generic connector, single row, 01x06, script generated"
 			(at 175.26 97.79 0)
-			(effects
-				(font
-					(size 1.27 1.27)
-				)
-				(hide yes)
+			(hide yes)
+			(show_name no)
+			(do_not_autoplace no)
+			(effects
+				(font
+					(size 1.27 1.27)
+				)
 			)
 		)
@@
 		)
 		(instances
-			(project ""
+			(project "PIEZO"
 				(path "/649320e7-4f25-4905-847f-0bb1c9cafdfd"
 					(reference "J1")
@@
 		(at 209.55 99.06 0)
 		(unit 1)
+		(body_style 1)
 		(exclude_from_sim no)
 		(in_bom yes)
 		(on_board yes)
+		(in_pos_files yes)
 		(dnp no)
 		(fields_autoplaced yes)
 		(property "Reference" "BZ1"
 			(at 213.36 97.7899 0)
+			(show_name no)
+			(do_not_autoplace no)
 			(effects
 				(font
@@
 		(property "Value" "Buzzer"
 			(at 213.36 100.3299 0)
+			(show_name no)
+			(do_not_autoplace no)
 			(effects
 				(font
@@
 		(property "Footprint" "PIEZO:buzzer"
 			(at 208.915 96.52 90)
-			(effects
-				(font
-					(size 1.27 1.27)
-				)
-				(hide yes)
-			)
-		)
-		(property "Datasheet" "~"
+			(hide yes)
+			(show_name no)
+			(do_not_autoplace no)
+			(effects
+				(font
+					(size 1.27 1.27)
+				)
+			)
+		)
+		(property "Datasheet" ""
 			(at 208.915 96.52 90)
-			(effects
-				(font
-					(size 1.27 1.27)
-				)
-				(hide yes)
+			(hide yes)
+			(show_name no)
+			(do_not_autoplace no)
+			(effects
+				(font
+					(size 1.27 1.27)
+				)
 			)
 		)
 		(property "Description" "Buzzer, polarized"
 			(at 209.55 99.06 0)
-			(effects
-				(font
-					(size 1.27 1.27)
-				)
-				(hide yes)
+			(hide yes)
+			(show_name no)
+			(do_not_autoplace no)
+			(effects
+				(font
+					(size 1.27 1.27)
+				)
 			)
 		)
@@
 		)
 		(instances
-			(project ""
+			(project "PIEZO"
 				(path "/649320e7-4f25-4905-847f-0bb1c9cafdfd"
 					(reference "BZ1")
@@
 		(at 203.2 96.52 90)
 		(unit 1)
+		(body_style 1)
 		(exclude_from_sim no)
 		(in_bom yes)
 		(on_board yes)
+		(in_pos_files yes)
 		(dnp no)
 		(fields_autoplaced yes)
 		(property "Reference" "R1"
 			(at 203.2 90.17 90)
+			(show_name no)
+			(do_not_autoplace no)
 			(effects
 				(font
@@
 		(property "Value" "330R"
 			(at 203.2 92.71 90)
+			(show_name no)
+			(do_not_autoplace no)
 			(effects
 				(font
@@
 		(property "Footprint" "Resistor_THT:R_Axial_DIN0207_L6.3mm_D2.5mm_P10.16mm_Horizontal"
 			(at 203.2 98.298 90)
-			(effects
-				(font
-					(size 1.27 1.27)
-				)
-				(hide yes)
-			)
-		)
-		(property "Datasheet" "~"
+			(hide yes)
+			(show_name no)
+			(do_not_autoplace no)
+			(effects
+				(font
+					(size 1.27 1.27)
+				)
+			)
+		)
+		(property "Datasheet" ""
 			(at 203.2 96.52 0)
-			(effects
-				(font
-					(size 1.27 1.27)
-				)
-				(hide yes)
+			(hide yes)
+			(show_name no)
+			(do_not_autoplace no)
+			(effects
+				(font
+					(size 1.27 1.27)
+				)
 			)
 		)
 		(property "Description" "Resistor"
 			(at 203.2 96.52 0)
-			(effects
-				(font
-					(size 1.27 1.27)
-				)
-				(hide yes)
+			(hide yes)
+			(show_name no)
+			(do_not_autoplace no)
+			(effects
+				(font
+					(size 1.27 1.27)
+				)
 			)
 		)
@@
 		)
 		(instances
-			(project ""
+			(project "PIEZO"
 				(path "/649320e7-4f25-4905-847f-0bb1c9cafdfd"
 					(reference "R1")

Commit message: Deployed 33ea02e with MkDocs version: 1.6.0
Parts:
- BZ1: value Buzzer -> PKHPS0013E4000-A2
Changed lines of the file:
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@@
 			)
 		)
-		(property "Value" "Buzzer"
+		(property "Value" "PKHPS0013E4000-A2"
 			(at 213.36 100.3299 0)
 			(show_name no)
