File: gyro/KiCad/akcelerometr2.kicad_pcb (KiCad board)
At the start: 2 copper layers, 16 x 37.5 mm, 5 parts, among them J2 Conn_01x04_Pin, J3 Conn_01x04_Pin, J4 Conn_01x08_Pin

Commit message: Deployed 0144617 with MkDocs version: 1.6.0
Parts:
- removed H1: MountingHole, MountingHole:MountingHole_3.2mm_M3
- removed J4: Conn_01x08_Pin, Connector_PinHeader_2.54mm:PinHeader_1x08_P2.54mm_Vertical
- added J1: Conn_01x06_Pin, Connector_PinHeader_2.54mm:PinHeader_1x06_P2.54mm_Horizontal, F.Cu at (109.0, 85.1)
- moved J3 24.9 mm to (125.4, 82.8)
- moved J2 24.5 mm to (125.4, 74.7)
- moved H2 21.8 mm to (117.3, 78.7)
Connections:
- net Net-(J2-Pin_3) renamed SDA
- net Net-(J2-Pin_4) renamed SCL
- net VCC renamed +3V3
Routing:
- net SDA: track 17.4 -> 25.7 mm
- net SCL: track 19.6 -> 25.9 mm, vias 0 -> 2
- net +3V3: track 24.8 -> 26.4 mm
- net GND: vias 11 -> 10
Other:
- board size 16 x 37.5 mm -> 24.4 x 17.3 mm
- board text added: "3V3"
- board text removed: "30mm"
- board text removed: "VCC"

Commit message: Deployed ba208f9 with MkDocs version: 1.6.0
Parts:
- removed J1: Conn_01x06_Pin, Connector_PinHeader_2.54mm:PinHeader_1x06_P2.54mm_Horizontal
- added H1: MountingHole, MountingHole:MountingHole_3.2mm_M3, F.Cu at (117.5, 69.0)
- added J4: Conn_01x08_Pin, Connector_PinHeader_2.54mm:PinHeader_1x08_P2.54mm_Horizontal, F.Cu at (109.0, 85.1)
Routing:
- net GND: vias 10 -> 12
Other:
- board size 24.4 x 17.3 mm -> 24.4 x 22.4 mm
- board text added: "H2"

Commit message: Deployed d972a79 with MkDocs version: 1.6.0
Parts:
- J4: value Conn_01x08_Pin -> Conn_01x06_Pin; footprint Connector_PinHeader_2.54mm:PinHeader_1x08_P2.54mm_Horizontal -> Connector_PinHeader_2.54mm:PinHeader_1x08_P2.54mm_Vertical
- moved J4 17.5 mm to (109.0, 67.6), turned to 0 degrees
- moved H2 4.80 mm to (118.0, 83.5)
- moved J3 2.28 mm to (125.5, 80.5)
- moved J2 2.20 mm to (125.5, 72.5)
- moved H1 0.71 mm to (118.0, 69.5)
Connections:
- J2 pad MP: (no net) -> GND
- J3 pad MP: (no net) -> GND
Routing:
- net +3V3: track 26.5 -> 28.8 mm, vias 0 -> 2
- net SDA: track 25.7 -> 24.8 mm, vias 2 -> 3
- net GND: vias 12 -> 21
Other:
- board size 24.4 x 22.4 mm -> 22 x 22 mm
- board text added: "20mm"
- board text added: "24mm"
- board text removed: "H2"
- board text removed: "M3"

Commit message: Deployed 2be6636 with MkDocs version: 1.6.0
Other:
- board text added: "22mm"
- board text removed: "20mm"
- board text removed: "24mm"
